File: hardware/seq1/neopxls.kicad_sch (KiCad schematic)
At the start: 11 parts, among them U11 Neopixel Keypad 1x4, U12 Neopixel Keypad 1x4, U13 Neopixel Keypad 1x4, U14 Neopixel Keypad 1x4, U2 74HC4051, U8 74HC4051

Commit message: Some schematic cleanup
Other:
- moved on the sheet: C18, C3, R7, TP2, TP4, U11, U12, U13, U14, U2, U8
