File: hardware/keypad_1x4/keypad_1x4.kicad_sch (KiCad schematic)
At the start: 11 parts, among them J1 Conn_01x04, J2 Conn_01x04, J3 Conn_01x01_Pin, J4 Conn_01x01_Pin, SW1 SW_Push_x4

Commit message: Some schematic cleanup
Parts:
- D1, D2, D3, D4: PN (none) -> IN-PI22TAT5R5G5B, Adafruit-3484
Changed lines of the file:
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@@
+			)
+		)
+		(property "PN" "IN-PI22TAT5R5G5B, Adafruit-3484"
+			(at 163.83 83.82 0)
+			(effects
+				(font
+					(size 1.27 1.27)
+				)
+				(hide yes)
 			)
 		)
@@
 			)
 		)
+		(property "PN" "IN-PI22TAT5R5G5B, Adafruit-3484"
+			(at 181.61 83.82 0)
+			(effects
+				(font
+					(size 1.27 1.27)
+				)
+				(hide yes)
+			)
+		)
 		(pin "1"
 		)
@@
 			)
 		)
+		(property "PN" "IN-PI22TAT5R5G5B, Adafruit-3484"
+			(at 146.05 83.82 0)
+			(effects
+				(font
+					(size 1.27 1.27)
+				)
+				(hide yes)
+			)
+		)
 		(pin "1"
 		)
@@
 			(at 128.27 83.82 0)
 			(effects
+				(font
+					(size 1.27 1.27)
+				)
+				(hide yes)
+			)
+		)
+		(property "PN" "IN-PI22TAT5R5G5B, Adafruit-3484"
+			(at 128.27 83.82 0)
+			(effects
